File: power.kicad_sch (KiCad schematic)
At the start: 44 parts, among them U10 74AUC2G32, U11 SN74AUP2G08, U12 74AUC2G32, U13 SN74AUP2G08, U14 74AUC2G32, U15 SN74AUP2G08, U16 SN74AUP2G08, U17 SN74AUP2G08, U18 74AUC2G32, U19 74AUC2G32, U20 SN74AUP2G08, U21 74AUC2G32, U22 SN74AUP2G08, U23 74AUC2G32, U24 SN74AUP2G08, U25 74AUC2G32, U26 SN74AUP2G08, U27 74AUC2G32, U28 SN74AUP2G08, U29 74AUC2G32, U8 SN74AUP2G08, U9 74AUC2G32

Commit message: schem: add ordering info to BOM
Parts:
- U10, U12, U14, U18, U19, U21, U23, U25, U27, U29, U9: Basic (none) -> X; JLCPCB Part # (none) -> C2876519; Manufacturer (none) -> Texas Instruments; Manufacturer Part Number (none) -> SN74AUP2G32DCUR
- U11, U13, U15, U16, U17, U20, U22, U24, U26, U28, U8: Basic (none) -> X; JLCPCB Part # (none) -> C544478; Manufacturer (none) -> Texas Instruments; Manufacturer Part Number (none) -> SN74AUP2G08DCUR

Commit message: schem: add title
Other:
- company: (none) -> Rémi Ait-Younes
- title: (none) -> DYB Segment Driver 1
Changed lines of the file:
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@@
 	(generator_version "10.0")
 	(paper "A4")
+	(title_block
+		(title "DYB Segment Driver 1")
+		(date "2026-09-29")
+		(rev "01")
+		(company "Rémi Ait-Younes")
+	)
 	(junction
 		(at 172.72 130.81)

Commit message: schem: reannotate
Parts:
- renumbered C22 to C10, C8 to C11, C16 to C12, C27 to C13, C9 to C14, C17 to C15, C28 to C16, C10 to C17, C29 to C19, C11 to C20, C19 to C21, C30 to C22, C12 to C23, C20 to C24, C31 to C25, C13 to C26, C21 to C27, C32 to C28, C14 to C29, C33 to C30, C15 to C9, U12 to U10, U14 to U11, U19 to U12, U18 to U13, U10 to U14, U20 to U17, U22 to U18, U24 to U19, U26 to U20, U28 to U21, U21 to U22, U25 to U24, U27 to U25, U29 to U26, U8 to U3, U11 to U4, U13 to U5, U15 to U6, U16 to U7, U17 to U8

Commit message: schem: fix footprints
Parts:
- U10, U11, U12, U13, U14, U22, U23, U24, U25, U26, U9: footprint Package_DFN_QFN:QFN-20-1EP_5x5mm_P0.65mm_EP3.35x3.35mm -> Package_SO:VSSOP-8_2.3x2mm_P0.5mm
Changed lines of the file:
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@@
 			)
 		)
-		(property "Footprint" "Package_DFN_QFN:QFN-20-1EP_5x5mm_P0.65mm_EP3.35x3.35mm"
+		(property "Footprint" "Package_SO:VSSOP-8_2.3x2mm_P0.5mm"
 			(at 182.88 53.34 0)
 			(hide yes)
@@
 			)
 		)
-		(property "Footprint" "Package_DFN_QFN:QFN-20-1EP_5x5mm_P0.65mm_EP3.35x3.35mm"
+		(property "Footprint" "Package_SO:VSSOP-8_2.3x2mm_P0.5mm"
 			(at 144.78 142.24 0)
 			(hide yes)
@@
 			)
 		)
-		(property "Footprint" "Package_DFN_QFN:QFN-20-1EP_5x5mm_P0.65mm_EP3.35x3.35mm"
+		(property "Footprint" "Package_SO:VSSOP-8_2.3x2mm_P0.5mm"
 			(at 127 53.34 0)
 			(hide yes)
@@
 			)
 		)
-		(property "Footprint" "Package_DFN_QFN:QFN-20-1EP_5x5mm_P0.65mm_EP3.35x3.35mm"
+		(property "Footprint" "Package_SO:VSSOP-8_2.3x2mm_P0.5mm"
 			(at 144.78 101.6 0)
 			(hide yes)
@@
 			)
 		)
-		(property "Footprint" "Package_DFN_QFN:QFN-20-1EP_5x5mm_P0.65mm_EP3.35x3.35mm"
+		(property "Footprint" "Package_SO:VSSOP-8_2.3x2mm_P0.5mm"
 			(at 172.72 142.24 0)
 			(hide yes)
@@
 			)
 		)
-		(property "Footprint" "Package_DFN_QFN:QFN-20-1EP_5x5mm_P0.65mm_EP3.35x3.35mm"
+		(property "Footprint" "Package_SO:VSSOP-8_2.3x2mm_P0.5mm"
 			(at 130.81 101.6 0)
 			(hide yes)
@@
 			)
 		)
-		(property "Footprint" "Package_DFN_QFN:QFN-20-1EP_5x5mm_P0.65mm_EP3.35x3.35mm"
+		(property "Footprint" "Package_SO:VSSOP-8_2.3x2mm_P0.5mm"
 			(at 116.84 142.24 0)
 			(hide yes)
@@
 			)
 		)
-		(property "Footprint" "Package_DFN_QFN:QFN-20-1EP_5x5mm_P0.65mm_EP3.35x3.35mm"
+		(property "Footprint" "Package_SO:VSSOP-8_2.3x2mm_P0.5mm"
 			(at 172.72 101.6 0)
 			(hide yes)
@@
 			)
 		)
-		(property "Footprint" "Package_DFN_QFN:QFN-20-1EP_5x5mm_P0.65mm_EP3.35x3.35mm"
+		(property "Footprint" "Package_SO:VSSOP-8_2.3x2mm_P0.5mm"
 			(at 154.94 53.34 0)
 			(hide yes)
@@
 			)
 		)
-		(property "Footprint" "Package_DFN_QFN:QFN-20-1EP_5x5mm_P0.65mm_EP3.35x3.35mm"
+		(property "Footprint" "Package_SO:VSSOP-8_2.3x2mm_P0.5mm"
 			(at 102.87 142.24 0)
 			(hide yes)
@@
 			)
 		)
-		(property "Footprint" "Package_DFN_QFN:QFN-20-1EP_5x5mm_P0.65mm_EP3.35x3.35mm"
+		(property "Footprint" "Package_SO:VSSOP-8_2.3x2mm_P0.5mm"
 			(at 113.03 53.34 0)
 			(hide yes)
